File: eurorack-synth.kicad_sch (KiCad schematic)
At the start: 5 parts

Commit message: Progress made
Parts:
- R?: value R -> 1K; footprint (none) -> Resistor_THT:R_Axial_DIN0204_L3.6mm_D1.6mm_P7.62mm_Horizontal
Connections:
- net GND: no longer D?.2 (A)
- net at J?.1 (Pin_1): now also D?.2 (A); no longer D?.1 (K)
- net at R?.2: now also D?.1 (K)
Other:
- moved on the sheet: D?
Changed lines of the file:
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@@
   (junction (at 233.68 127) (diameter 0) (color 0 0 0 0)
   )
-  (wire (pts (xy 86.36 115.57) (xy 86.36 118.11))
-    (stroke (width 0) (type default) (color 0 0 0 0))
-  )
-  (wire (pts (xy 100.33 115.57) (xy 86.36 115.57))
-    (stroke (width 0) (type default) (color 0 0 0 0))
-  )
   (wire (pts (xy 97.79 118.11) (xy 100.33 118.11))
     (stroke (width 0) (type default) (color 0 0 0 0))
@@
     (stroke (width 0) (type default) (color 0 0 0 0))
   )
-  (wire (pts (xy 86.36 125.73) (xy 86.36 128.27))
-    (stroke (width 0) (type default) (color 0 0 0 0))
-  )
   (wire (pts (xy 114.3 77.47) (xy 114.3 81.28))
     (stroke (width 0) (type default) (color 0 0 0 0))
@@
     (stroke (width 0) (type default) (color 0 0 0 0))
   )
+  (wire (pts (xy 96.52 115.57) (xy 100.33 115.57))
+    (stroke (width 0) (type default) (color 0 0 0 0))
+  )
   (wire (pts (xy 127 95.25) (xy 127 100.33))
     (stroke (width 0) (type default) (color 0 0 0 0))
   )
   (wire (pts (xy 134.62 102.87) (xy 134.62 100.33))
+    (stroke (width 0) (type default) (color 0 0 0 0))
+  )
+  (wire (pts (xy 83.82 115.57) (xy 88.9 115.57))
     (stroke (width 0) (type default) (color 0 0 0 0))
   )
@@
     (pin "2")
   )
-  (symbol (lib_id "Diode:1N4001") (at 86.36 121.92 270) (unit 1)
-    (in_bom yes) (on_board yes) (fields_autoplaced)
-    (property "Reference" "D?" (id 0) (at 88.9 120.6499 90)
-      (effects (font (size 1.27 1.27)) (justify left))
-    )
-    (property "Value" "1N4001" (id 1) (at 88.9 123.1899 90)
-      (effects (font (size 1.27 1.27)) (justify left))
-    )
-    (property "Footprint" "Diode_THT:D_DO-41_SOD81_P10.16mm_Horizontal" (id 2) (at 81.915 121.92 0)
-      (effects (font (size 1.27 1.27)) hide)
-    )
-    (property "Datasheet" "http://www.vishay.com/docs/88503/1n4001.pdf" (id 3) (at 86.36 121.92 0)
+  (symbol (lib_id "Diode:1N4001") (at 92.71 115.57 0) (unit 1)
+    (in_bom yes) (on_board yes) (fields_autoplaced)
+    (property "Reference" "D?" (id 0) (at 92.71 109.22 0))
+    (property "Value" "1N4001" (id 1) (at 92.71 111.76 0))
+    (property "Footprint" "Diode_THT:D_DO-41_SOD81_P10.16mm_Horizontal" (id 2) (at 92.71 120.015 0)
+      (effects (font (size 1.27 1.27)) hide)
+    )
+    (property "Datasheet" "http://www.vishay.com/docs/88503/1n4001.pdf" (id 3) (at 92.71 115.57 0)
       (effects (font (size 1.27 1.27)) hide)
     )
@@
     (in_bom yes) (on_board yes) (fields_autoplaced)
     (property "Reference" "R?" (id 0) (at 80.01 109.22 90))
-    (property "Value" "R" (id 1) (at 80.01 111.76 90))
-    (property "Footprint" "" (id 2) (at 80.01 117.348 90)
+    (property "Value" "1K" (id 1) (at 80.01 111.76 90))
+    (property "Footprint" "Resistor_THT:R_Axial_DIN0204_L3.6mm_D1.6mm_P7.62mm_Horizontal" (id 2) (at 80.01 117.348 90)
       (effects (font (size 1.27 1.27)) hide)
     )
@@
     (pin "TP6")
   )
-  (symbol (lib_id "power:GND") (at 86.36 128.27 0) (unit 1)
-    (in_bom yes) (on_board yes) (fields_autoplaced)
-    (property "Reference" "#PWR?" (id 0) (at 86.36 134.62 0)
-      (effects (font (size 1.27 1.27)) hide)
-    )
-    (property "Value" "GND" (id 1) (at 86.36 133.35 0))
-    (property "Footprint" "" (id 2) (at 86.36 128.27 0)
-      (effects (font (size 1.27 1.27)) hide)
-    )
-    (property "Datasheet" "" (id 3) (at 86.36 128.27 0)
-      (effects (font (size 1.27 1.27)) hide)
-    )
-    (pin "1")
-  )
   (symbol (lib_id "power:GND") (at 127 100.33 0) (unit 1)
     (in_bom yes) (on_board yes) (fields_autoplaced)
@@
       (reference "#PWR?") (unit 1) (value "+3V3") (footprint "")
     )
-    (path "/c5adbd49-cdfd-47c6-8f9f-eadceb2a44be"
-      (reference "#PWR?") (unit 1) (value "GND") (footprint "")
-    )
     (path "/d2430afd-9d1b-4678-bd3d-aae6923d00ed"
       (reference "#PWR?") (unit 1) (value "GND") (footprint "")
@@
     )
     (path "/942a8977-afdd-4763-804f-2a3f20694e8f"
-      (reference "R?") (unit 1) (value "R") (footprint "")
+      (reference "R?") (unit 1) (value "1K") (footprint "Resistor_THT:R_Axial_DIN0204_L3.6mm_D1.6mm_P7.62mm_Horizontal")
     )
     (path "/311764c7-b652-45a2-af0b-30d0ba8793a5"

Commit message: Made some progress
Parts:
- added J?: Gate, symbol Connector:Conn_01x02_Female
- added R?: 3K3, Resistor_THT:R_Axial_DIN0204_L3.6mm_D1.6mm_P7.62mm_Horizontal, symbol Device:R
- added R?: 1K, Resistor_THT:R_Axial_DIN0204_L3.6mm_D1.6mm_P7.62mm_Horizontal, symbol Device:R
- added RV?: R_Potentiometer, symbol Device:R_Potentiometer
- J?: value Conn_01x02_Female -> Pitch CV
Connections:
- net GND: now also J?.2 (Pin_2), R?.1
- net Gate: now reaches U?.29 (GP22)
- net Gate: now also R?.2, R?.2
- new net: J?.1 (Pin_1), R?.1
Changed lines of the file:
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@@
   (junction (at 233.68 127) (diameter 0) (color 0 0 0 0)
   )
+  (wire (pts (xy 146.05 173.99) (xy 143.51 173.99))
+    (stroke (width 0) (type default) (color 0 0 0 0))
+  )
   (wire (pts (xy 97.79 118.11) (xy 100.33 118.11))
     (stroke (width 0) (type default) (color 0 0 0 0))
@@
     (stroke (width 0) (type default) (color 0 0 0 0))
   )
+  (wire (pts (xy 160.02 176.53) (xy 157.48 176.53))
+    (stroke (width 0) (type default) (color 0 0 0 0))
+  )
   (wire (pts (xy 97.79 120.65) (xy 97.79 118.11))
     (stroke (width 0) (type default) (color 0 0 0 0))
@@
     (stroke (width 0) (type default) (color 0 0 0 0))
   )
+  (wire (pts (xy 153.67 173.99) (xy 160.02 173.99))
+    (stroke (width 0) (type default) (color 0 0 0 0))
+  )
   (wire (pts (xy 96.52 115.57) (xy 100.33 115.57))
     (stroke (width 0) (type default) (color 0 0 0 0))
   )
+  (wire (pts (xy 143.51 184.15) (xy 143.51 186.69))
+    (stroke (width 0) (type default) (color 0 0 0 0))
+  )
   (wire (pts (xy 127 95.25) (xy 127 100.33))
     (stroke (width 0) (type default) (color 0 0 0 0))
@@
     (stroke (width 0) (type default) (color 0 0 0 0))
   )
+  (wire (pts (xy 143.51 173.99) (xy 143.51 176.53))
+    (stroke (width 0) (type default) (color 0 0 0 0))
+  )
   (wire (pts (xy 83.82 115.57) (xy 88.9 115.57))
     (stroke (width 0) (type default) (color 0 0 0 0))
@@
     (stroke (width 0) (type default) (color 0 0 0 0))
   )
+  (wire (pts (xy 157.48 176.53) (xy 157.48 179.07))
+    (stroke (width 0) (type default) (color 0 0 0 0))
+  )
   (label "A" (at 233.68 91.44 0)
     (effects (font (size 1.27 1.27)) (justify left bottom))
+  )
+  (label "Gate" (at 143.51 173.99 180)
+    (effects (font (size 1.27 1.27)) (justify right bottom))
   )
   (label "release" (at 142.24 82.55 0)
@@
     (effects (font (size 1.27 1.27)) (justify left bottom))
   )
+  (label "Gate" (at 233.68 88.9 0)
+    (effects (font (size 1.27 1.27)) (justify left bottom))
+  )
   (label "S2" (at 116.84 67.31 180)
     (effects (font (size 1.27 1.27)) (justify right bottom))
@@
     (effects (font (size 1.27 1.27)) (justify right bottom))
   )
+  (symbol (lib_id "power:GND") (at 143.51 186.69 0) (unit 1)
+    (in_bom yes) (on_board yes) (fields_autoplaced)
+    (property "Reference" "#PWR?" (id 0) (at 143.51 193.04 0)
+      (effects (font (size 1.27 1.27)) hide)
+    )
+    (property "Value" "GND" (id 1) (at 143.51 191.77 0))
+    (property "Footprint" "" (id 2) (at 143.51 186.69 0)
+      (effects (font (size 1.27 1.27)) hide)
+    )
+    (property "Datasheet" "" (id 3) (at 143.51 186.69 0)
+      (effects (font (size 1.27 1.27)) hide)
+    )
+    (pin "1")
+  )
   (symbol (lib_id "power:GND") (at 97.79 120.65 0) (unit 1)
     (in_bom yes) (on_board yes) (fields_autoplaced)
@@
     )
     (property "Datasheet" "" (id 3) (at 240.03 132.08 0)
+      (effects (font (size 1.27 1.27)) hide)
+    )
+    (pin "1")
+  )
+  (symbol (lib_id "power:GND") (at 157.48 179.07 0) (unit 1)
+    (in_bom yes) (on_board yes) (fields_autoplaced)
+    (property "Reference" "#PWR?" (id 0) (at 157.48 185.42 0)
+      (effects (font (size 1.27 1.27)) hide)
+    )
+    (property "Value" "GND" (id 1) (at 157.48 184.15 0))
+    (property "Footprint" "" (id 2) (at 157.48 179.07 0)
+      (effects (font (size 1.27 1.27)) hide)
+    )
+    (property "Datasheet" "" (id 3) (at 157.48 179.07 0)
       (effects (font (size 1.27 1.27)) hide)
     )
@@
       (effects (font (size 1.27 1.27)) (justify left))
     )
-    (property "Value" "Conn_01x02_Female" (id 1) (at 106.68 118.1099 0)
+    (property "Value" "Pitch CV" (id 1) (at 106.68 118.1099 0)
       (effects (font (size 1.27 1.27)) (justify left))
     )
@@
     (pin "1")
     (pin "2")
+  )
+  (symbol (lib_id "Device:R_Potentiometer") (at 81.28 130.81 0) (unit 1)
+    (in_bom yes) (on_board yes) (fields_autoplaced)
+    (property "Reference" "RV?" (id 0) (at 78.74 129.5399 0)
+      (effects (font (size 1.27 1.27)) (justify right))
+    )
+    (property "Value" "R_Potentiometer" (id 1) (at 78.74 132.0799 0)
+      (effects (font (size 1.27 1.27)) (justify right))
+    )
+    (property "Footprint" "" (id 2) (at 81.28 130.81 0)
+      (effects (font (size 1.27 1.27)) hide)
+    )
+    (property "Datasheet" "~" (id 3) (at 81.28 130.81 0)
+      (effects (font (size 1.27 1.27)) hide)
+    )
+    (pin "1")
+    (pin "2")
+    (pin "3")
   )
   (symbol (lib_id "Diode:1N4001") (at 92.71 115.57 0) (unit 1)
@@
     (pin "TP6")
   )
+  (symbol (lib_id "Device:R") (at 143.51 180.34 180) (unit 1)
+    (in_bom yes) (on_board yes) (fields_autoplaced)
+    (property "Reference" "R?" (id 0) (at 146.05 179.0699 0)
+      (effects (font (size 1.27 1.27)) (justify right))
+    )
+    (property "Value" "3K3" (id 1) (at 146.05 181.6099 0)
+      (effects (font (size 1.27 1.27)) (justify right))
+    )
+    (property "Footprint" "Resistor_THT:R_Axial_DIN0204_L3.6mm_D1.6mm_P7.62mm_Horizontal" (id 2) (at 145.288 180.34 90)
+      (effects (font (size 1.27 1.27)) hide)
+    )
+    (property "Datasheet" "~" (id 3) (at 143.51 180.34 0)
+      (effects (font (size 1.27 1.27)) hide)
+    )
+    (pin "1")
+    (pin "2")
+  )
   (symbol (lib_id "power:GND") (at 127 100.33 0) (unit 1)
     (in_bom yes) (on_board yes) (fields_autoplaced)
@@
     (pin "1")
   )
+  (symbol (lib_id "Device:R") (at 149.86 173.99 270) (unit 1)
+    (in_bom yes) (on_board yes) (fields_autoplaced)
+    (property "Reference" "R?" (id 0) (at 149.86 167.64 90))
+    (property "Value" "1K" (id 1) (at 149.86 170.18 90))
+    (property "Footprint" "Resistor_THT:R_Axial_DIN0204_L3.6mm_D1.6mm_P7.62mm_Horizontal" (id 2) (at 149.86 172.212 90)
+      (effects (font (size 1.27 1.27)) hide)
+    )
+    (property "Datasheet" "~" (id 3) (at 149.86 173.99 0)
+      (effects (font (size 1.27 1.27)) hide)
+    )
+    (pin "1")
+    (pin "2")
+  )
+  (symbol (lib_id "Connector:Conn_01x02_Female") (at 165.1 173.99 0) (unit 1)
+    (in_bom yes) (on_board yes) (fields_autoplaced)
+    (property "Reference" "J?" (id 0) (at 166.37 173.9899 0)
+      (effects (font (size 1.27 1.27)) (justify left))
+    )
+    (property "Value" "Gate" (id 1) (at 166.37 176.5299 0)
+      (effects (font (size 1.27 1.27)) (justify left))
+    )
+    (property "Footprint" "" (id 2) (at 165.1 173.99 0)
+      (effects (font (size 1.27 1.27)) hide)
+    )
+    (property "Datasheet" "~" (id 3) (at 165.1 173.99 0)
+      (effects (font (size 1.27 1.27)) hide)
+    )
+    (pin "1")
+    (pin "2")
+  )
   (sheet_instances
     (path "/" (page "1"))
   )
   (symbol_instances
+    (path "/03fafb79-e9b4-46d8-a707-df52bba50ac0"
+      (reference "#PWR?") (unit 1) (value "GND") (footprint "")
+    )
     (path "/0e9f4d17-ca75-486d-a338-34ac220e0419"
       (reference "#PWR?") (unit 1) (value "GND") (footprint "")
@@
     )
     (path "/1c135714-1d6d-401b-a2f5-75689263311d"
+      (reference "#PWR?") (unit 1) (value "GND") (footprint "")
+    )
+    (path "/2e82f573-84c7-4545-ae28-f9e6f082319e"
       (reference "#PWR?") (unit 1) (value "GND") (footprint "")
     )
@@
     )
     (path "/34d106b4-0117-4a71-b27c-8f44bcde1aa5"
-      (reference "J?") (unit 1) (value "Conn_01x02_Female") (footprint "")
+      (reference "J?") (unit 1) (value "Pitch CV") (footprint "")
+    )
+    (path "/f5bf0ae3-d365-4548-8580-8061d71f1037"
+      (reference "J?") (unit 1) (value "Gate") (footprint "")
     )
     (path "/942a8977-afdd-4763-804f-2a3f20694e8f"
       (reference "R?") (unit 1) (value "1K") (footprint "Resistor_THT:R_Axial_DIN0204_L3.6mm_D1.6mm_P7.62mm_Horizontal")
     )
+    (path "/c262f517-002c-4048-9f64-bf4db62625b4"
+      (reference "R?") (unit 1) (value "3K3") (footprint "Resistor_THT:R_Axial_DIN0204_L3.6mm_D1.6mm_P7.62mm_Horizontal")
+    )
+    (path "/f1cb2f29-c0cd-4c01-b649-68c2dbee9f2b"
+      (reference "R?") (unit 1) (value "1K") (footprint "Resistor_THT:R_Axial_DIN0204_L3.6mm_D1.6mm_P7.62mm_Horizontal")
+    )
+    (path "/849280c8-0991-4775-a8b6-0a3032c9e3df"
+      (reference "RV?") (unit 1) (value "R_Potentiometer") (footprint "")
+    )
     (path "/311764c7-b652-45a2-af0b-30d0ba8793a5"
